File: Hardware/op_board/op_board.kicad_sch (KiCad schematic)
At the start: 80 parts, among them J1 Conn_01x01, J10 Conn_01x01, J11 Conn_01x04, J12 Conn_01x01, J13 Conn_01x01, J14 Conn_01x01, J15 Conn_01x01, J16 Conn_01x01, J17 Conn_01x01, J18 Conn_01x01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

Commit message: small updates change to Kicad V7
Parts:
- removed TP16, TP17, TP18, TP2: RCWCTE, MyLib:TP420X150, symbol MyLib:RCWCTE
- TP1, TP10, TP11, TP12, TP13, TP14, TP15, TP19, TP20, TP3, TP4, TP5, TP6, TP7, TP8, TP9: footprint MyLib:TP420X150 -> TP420X150
