File: Hardware/op_board/op_board.kicad_pcb (KiCad board)
At the start: 2 copper layers, 58.1 x 63.1 mm, 76 parts, among them J1 Conn_01x01, J10 Conn_01x01, J11 Conn_01x04, J12 Conn_01x01, J13 Conn_01x01, J14 Conn_01x01, J15 Conn_01x01, J16 Conn_01x01, J17 Conn_01x01, J18 Conn_01x01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

Commit message: small updates change to Kicad V7
Parts:
- moved TP6 0.25 mm to (144.8, 151.4), turned to 0 degrees

Commit message: small updates, files used for order
Other:
- board text added: "OUT"
Changed lines of the file:
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@@
     (property "ki_keywords" "connector")
     (attr exclude_from_pos_files)
-    (fp_text reference "J10" (at -2.894 -1.1484) (layer "F.SilkS")
+    (fp_text reference "J10" (at -2.894 -1.1484) (layer "F.SilkS") hide
         (effects (font (size 1 1) (thickness 0.15)))
     )
@@
     (property "ki_keywords" "connector")
     (attr exclude_from_pos_files)
-    (fp_text reference "J9" (at 0 2.54) (layer "F.SilkS")
+    (fp_text reference "J9" (at 0 2.54) (layer "F.SilkS") hide
         (effects (font (size 1 1) (thickness 0.15)))
     )
@@
     (effects (font (size 1 1) (thickness 0.15)))
   )
+  (gr_text "OUT\n" (at 150 152) (layer "F.SilkS")
+    (effects (font (size 1 1) (thickness 0.15)) (justify left bottom))
+  )
   (gr_text "V+ GND  V-\n" (at 152.908 137.668 90) (layer "F.SilkS")
     (effects (font (size 1.5 1.4) (thickness 0.15)))
@@
     (effects (font (size 1 1) (thickness 0.15)))
   )
+  (gr_text "OUT\n" (at 148 117) (layer "F.SilkS")
+    (effects (font (size 1 1) (thickness 0.15)) (justify left bottom))
+  )
   (gr_text "Ref-  IN-    IN+   Ref+" (at 98.5 154.5 -90) (layer "F.SilkS")
